Commit message: add wheel params in launches

File: panther_description/urdf/panther.urdf.xacro (robot description, xacro)
@@ -11,5 +11,7 @@
   <xacro:arg name="imu_rot_y" default="-1.57" />
   <xacro:arg name="simulation_engine" default="ignition-gazebo" />
-  <xacro:arg name="controllers_config_file"
+  <xacro:arg name="wheel_config_file"
+    default="$(find panther_description)/config/WH01.yaml" />
+  <xacro:arg name="controller_config_file"
     default="$(find panther_controller)/config/WH01_controller.yaml" />
   <xacro:include filename="$(find panther_description)/urdf/panther_macro.urdf.xacro" ns="husarion" />
@@ -24,4 +26,5 @@
     imu_rot_y="$(arg imu_rot_y)"
     simulation_engine="$(arg simulation_engine)"
-    controllers_config_file="$(arg controllers_config_file)"/>
+    wheel_config_file="$(arg wheel_config_file)"
+    controller_config_file="$(arg controller_config_file)"/>
 </robot>

File: panther_description/urdf/panther_macro.urdf.xacro (robot description, xacro)
@@ -3,5 +3,6 @@
   <xacro:macro
     name="panther_robot"
-    params="controllers_config_file
+    params="wheel_config_file
+            controller_config_file
             use_sim:=false
             dual_bat:=false
@@ -13,6 +14,7 @@
             imu_rot_y:=0.0
             simulation_engine:='ignition-gazebo'">
-    <xacro:property name="controllers_config" value="${xacro.load_yaml(controllers_config_file)}" />
-    <xacro:property name="wheel_config" value="${controllers_config['wheel_params']['ros__parameters']}" />
+    <xacro:property name="wheel_config" value="${xacro.load_yaml(wheel_config_file)}" />
+    <xacro:property name="controllers_config" value="${xacro.load_yaml(controller_config_file)}" />
+    <xacro:property name="wheel_separation_x" value="0.44" />
     <!-- INCLUDE ROBOT PARTS DEFINITIONS -->
     <xacro:include filename="$(find panther_description)/urdf/body.urdf.xacro" ns="body" />
@@ -28,5 +30,4 @@
       imu_rot_y="${imu_rot_y}"
       simulation_engine="${simulation_engine}" />
-    <xacro:property name="wheel_separation_x" value="0.44" />
     <!-- WHEEL DECLARATION -->
     <xacro:wheel.wheel
@@ -110,5 +111,5 @@
         <plugin filename="ign_ros2_control-system"
           name="ign_ros2_control::IgnitionROS2ControlPlugin">
-          <parameters>${controllers_config_file}</parameters>
+          <parameters>${controller_config_file}</parameters>
           <ros>
             <remapping>/panther_base_controller/cmd_vel_unstamped:=/cmd_vel</remapping>
@@ -116,11 +117,25 @@
         </plugin>
       </gazebo>
+      <gazebo>
+        <plugin filename="ignition-gazebo-linearbatteryplugin-system"
+          name="gz::sim::systems::LinearBatteryPlugin">
+          <battery_name>panther_battery</battery_name>
+          <voltage>42</voltage>
+          <open_circuit_voltage_constant_coef>42</open_circuit_voltage_constant_coef>
+          <open_circuit_voltage_linear_coef>-10.0</open_circuit_voltage_linear_coef>
+          <initial_charge>20</initial_charge>
+          <capacity>20 </capacity>
+          <resistance>0.15</resistance>
+          <smooth_current_tau>2.0</smooth_current_tau>
+          <enable_recharge>true</enable_recharge>
+          <charging_time>6.0</charging_time>
+          <soc_threshold>2</soc_threshold>
+          <power_load>25</power_load>
+          <start_on_motion>false</start_on_motion>
+        </plugin>
+      </gazebo>
       <gazebo reference="imu_link">
         <sensor name="imu" type="imu">
-          <plugin filename="ignition-gazebo-imu-system" name="ignition::gazebo::systems::Imu">
-            <ros>
-              <remapping>/imu_broadcaster/imu:=/imu/data_raw</remapping>
-            </ros>
-          </plugin>
+          <plugin filename="ignition-gazebo-imu-system" name="ignition::gazebo::systems::Imu" />
           <always_on>true</always_on>
           <update_rate>100</update_rate>

File: panther_description/urdf/wheel.urdf.xacro (robot description, xacro)
@@ -3,6 +3,4 @@
   <!-- wheel defining macro -->
   <xacro:macro name="wheel" params="wheel_config wheel_separation_x prefix">
-    <xacro:property name="max_lin_velocity" value="2.0" />
-    <xacro:property name="max_ang_velocity" value="${max_lin_velocity / wheel_config['wheel_radius']}" />
     <xacro:if value="${prefix == 'fl'}">
       <xacro:property name="x" value="${wheel_separation_x/2.0}" />
@@ -30,5 +28,5 @@
       <child link="${prefix}_wheel_link" />
       <axis xyz="0.0 1.0 0.0" />
-      <limit effort="34.5" velocity="${max_ang_velocity}" />
+      <limit effort="34.5" velocity="10.958" />
       <dynamics damping="0.01" friction="0.01" />
     </joint>

Commit message: add battery plugin

File: panther_description/urdf/panther.urdf.xacro (robot description, xacro)
@@ -3,5 +3,4 @@
   <xacro:arg name="use_sim" default="false" />
   <xacro:arg name="use_gpu" default="false" />
-  <xacro:arg name="dual_bat" default="false" />
   <xacro:arg name="imu_pos_x" default="0.169" />
   <xacro:arg name="imu_pos_y" default="0.025" />
@@ -15,8 +14,9 @@
   <xacro:arg name="controller_config_file"
     default="$(find panther_controller)/config/WH01_controller.yaml" />
+  <xacro:arg name="battery_config_file"
+    default="$(find panther_description)/config/battery_ign_plugin.yaml" />
   <xacro:include filename="$(find panther_description)/urdf/panther_macro.urdf.xacro" ns="husarion" />
   <xacro:husarion.panther_robot
     use_sim="$(arg use_sim)"
-    dual_bat="$(arg dual_bat)"
     imu_pos_x="$(arg imu_pos_x)"
     imu_pos_y="$(arg imu_pos_y)"
@@ -27,4 +27,5 @@
     simulation_engine="$(arg simulation_engine)"
     wheel_config_file="$(arg wheel_config_file)"
-    controller_config_file="$(arg controller_config_file)"/>
+    controller_config_file="$(arg controller_config_file)"
+    battery_config_file="$(arg battery_config_file)" />
 </robot>

File: panther_description/urdf/panther_macro.urdf.xacro (robot description, xacro)
@@ -5,6 +5,6 @@
     params="wheel_config_file
             controller_config_file
+            battery_config_file
             use_sim:=false
-            dual_bat:=false
             imu_pos_x:=0.168
             imu_pos_y:=0.028
@@ -16,4 +16,16 @@
     <xacro:property name="wheel_config" value="${xacro.load_yaml(wheel_config_file)}" />
     <xacro:property name="controllers_config" value="${xacro.load_yaml(controller_config_file)}" />
+    <xacro:if value="${use_sim}">
+      <xacro:property name="battery_config" value="${xacro.load_yaml(battery_config_file)}" />
+      <xacro:property name="bat_initial_charge"
+        value="${20*battery_config['initial_charge_percentage']/100.0}" />
+      <xacro:property name="bat_charging_time" value="${battery_config['charging_time']}" />
+      <xacro:if value="${battery_config['simulate_discharging']}">
+        <xacro:property name="bat_power_load" value="${battery_config['power_load']}" />
+      </xacro:if>
+      <xacro:unless value="${battery_config['simulate_discharging']}">
+        <xacro:property name="bat_power_load" value="0.0" />
+      </xacro:unless>
+    </xacro:if>
     <xacro:property name="wheel_separation_x" value="0.44" />
     <!-- INCLUDE ROBOT PARTS DEFINITIONS -->
@@ -124,13 +136,15 @@
           <open_circuit_voltage_constant_coef>42</open_circuit_voltage_constant_coef>
           <open_circuit_voltage_linear_coef>-10.0</open_circuit_voltage_linear_coef>
-          <initial_charge>20</initial_charge>
+          <initial_charge>${bat_initial_charge}</initial_charge>
           <capacity>20 </capacity>
           <resistance>0.15</resistance>
           <smooth_current_tau>2.0</smooth_current_tau>
           <enable_recharge>true</enable_recharge>
-          <charging_time>6.0</charging_time>
-          <soc_threshold>2</soc_threshold>
-          <power_load>25</power_load>
+          <charging_time>${bat_charging_time}</charging_time>
+          <soc_threshold>2.0</soc_threshold>
+          <power_load>${bat_power_load}</power_load>
           <start_on_motion>false</start_on_motion>
+          <!-- https://github.com/gazebosim/gz-sim/issues/225 -->
+          <fix_issue_225>true</fix_issue_225>
         </plugin>
       </gazebo>
