Commit message: Update panther_description/urdf/panther_macro.urdf.xacro
Co-authored-by: Dawid Kmak <73443304+KmakD@users.noreply.github.com>

File: panther_description/urdf/panther_macro.urdf.xacro (robot description, xacro)
@@ -15,5 +15,4 @@
             simulation_engine:='ignition-gazebo'">
     <xacro:property name="wheel_config" value="${xacro.load_yaml(wheel_config_file)}" />
-    <xacro:property name="controllers_config" value="${xacro.load_yaml(controller_config_file)}" />
     <xacro:if value="${use_sim}">
       <xacro:property name="battery_config" value="${xacro.load_yaml(battery_config_file)}" />
