Commit message: add mesh path parsing

File: panther_description/urdf/body.urdf.xacro (robot description, xacro)
@@ -18,5 +18,5 @@
         <origin xyz="0.0 0.0 0.0" rpy="0.0 0.0 0.0" />
         <geometry>
-          <mesh filename="file://$(find panther_description)/meshes/body.dae" />
+          <mesh filename="package://panther_description/meshes/body.dae" />
         </geometry>
       </visual>
@@ -24,5 +24,5 @@
         <origin xyz="0.0 0.0 0.0" rpy="0.0 0.0 0.0" />
         <geometry>
-          <mesh filename="file://$(find panther_description)/meshes/body_collision.stl" />
+          <mesh filename="package://panther_description/meshes/body_collision.stl" />
         </geometry>
       </collision>

File: panther_description/urdf/components/external_antenna.urdf.xacro (robot description, xacro)
@@ -27,5 +27,5 @@
         <origin xyz="0.0 0.0 0.0" rpy="0.0 0.0 0.0" />
         <geometry>
-          <mesh filename="file://$(find panther_description)/meshes/components/external_antenna.dae" />
+          <mesh filename="package://panther_description/meshes/components/external_antenna.dae" />
         </geometry>
       </visual>
@@ -34,5 +34,5 @@
         <geometry>
           <mesh
-            filename="file://$(find panther_description)/meshes/components/external_antenna_collision.stl" />
+            filename="package://panther_description/meshes/components/external_antenna_collision.stl" />
         </geometry>
       </collision>

File: panther_description/urdf/wheel.urdf.xacro (robot description, xacro)
@@ -7,4 +7,5 @@
       <xacro:property name="y" value="${wheel_config['wheel_separation']/2.0}" />
       <xacro:property name="inertia_y_offset" value="${wheel_config['inertia_y_offset']}" />
+      <xacro:property name="fdir" value="1 -1 0" />
     </xacro:if>
     <xacro:if value="${prefix == 'fr'}">
@@ -12,4 +13,5 @@
       <xacro:property name="y" value="-${wheel_config['wheel_separation']/2.0}" />
       <xacro:property name="inertia_y_offset" value="${-wheel_config['inertia_y_offset']}" />
+      <xacro:property name="fdir" value="1 1 0" />
     </xacro:if>
     <xacro:if value="${prefix == 'rl'}">
@@ -17,4 +19,5 @@
       <xacro:property name="y" value="${wheel_config['wheel_separation']/2.0}" />
       <xacro:property name="inertia_y_offset" value="${wheel_config['inertia_y_offset']}" />
+      <xacro:property name="fdir" value="1 1 0" />
     </xacro:if>
     <xacro:if value="${prefix == 'rr'}">
@@ -22,4 +25,5 @@
       <xacro:property name="y" value="-${wheel_config['wheel_separation']/2.0}" />
       <xacro:property name="inertia_y_offset" value="${-wheel_config['inertia_y_offset']}" />
+      <xacro:property name="fdir" value="1 -1 0" />
     </xacro:if>
     <joint name="${prefix}_wheel_joint" type="continuous">
@@ -28,5 +32,5 @@
       <child link="${prefix}_wheel_link" />
       <axis xyz="0.0 1.0 0.0" />
-      <limit effort="34.5" velocity="10.958" />
+      <limit effort="64.5" velocity="10.958" />
       <dynamics damping="0.01" friction="0.01" />
     </joint>
@@ -36,5 +40,5 @@
         <geometry>
           <mesh
-            filename="file://$(find ${wheel_config['mesh_package']})/${wheel_config['folder_path']}/${prefix}_wheel.dae" />
+            filename="package://${wheel_config['mesh_package']}/${wheel_config['folder_path']}/${prefix}_wheel.dae" />
         </geometry>
       </visual>
@@ -43,5 +47,5 @@
         <geometry>
           <mesh
-            filename="file://$(find ${wheel_config['mesh_package']})/${wheel_config['folder_path']}/wheel_collision.stl" />
+            filename="package://${wheel_config['mesh_package']}/${wheel_config['folder_path']}/wheel_collision.stl" />
         </geometry>
       </collision>
@@ -58,4 +62,19 @@
       </inertial>
     </link>
+    <xacro:if value="${use_sim}">
+      <gazebo reference="${prefix}_wheel_link" xmlns:ignition="http://ignitionrobotics.org/schema">
+        <collision>
+          <surface>
+            <friction>
+              <ode>
+                <mu>1.0</mu>
+                <mu2>0.0</mu2>
+                <fdir1 ignition:expressed_in="base_link">${fdir}</fdir1>
+              </ode>
+            </friction>
+          </surface>
+        </collision>
+      </gazebo>
+    </xacro:if>
   </xacro:macro>
 </robot>

Commit message: review fixes

File: panther_description/urdf/body.urdf.xacro (robot description, xacro)
@@ -5,5 +5,4 @@
     name="body"
     params="wheel_radius
-            simulation_engine
             imu_pos_x imu_pos_y imu_pos_z
             imu_rot_r imu_rot_p imu_rot_y">
@@ -42,13 +41,25 @@
     </joint>
     <link name="imu_link" />
-    <joint name="body_to_front_light_joint" type="fixed">
+    <joint name="body_to_front_bumper_joint" type="fixed">
       <origin xyz="0.362 0.0 0.0" rpy="0.0 0.0 0.0" />
       <parent link="body_link" />
+      <child link="front_bumper_link" />
+    </joint>
+    <link name="front_bumper_link" />
+    <joint name="front_bumper_to_front_light_joint" type="fixed">
+      <origin xyz="0.0 0.0 0.0185" rpy="${pi/2} 0.0 ${pi/2}" />
+      <parent link="front_bumper_link" />
       <child link="front_light_link" />
     </joint>
     <link name="front_light_link" />
-    <joint name="body_to_rear_light_joint" type="fixed">
+    <joint name="body_to_rear_bumper_joint" type="fixed">
       <origin xyz="-0.362 0.0 0.0" rpy="0.0 0.0 ${pi}" />
       <parent link="body_link" />
+      <child link="rear_bumper_link" />
+    </joint>
+    <link name="rear_bumper_link" />
+    <joint name="rear_bumper_to_rear_light_joint" type="fixed">
+      <origin xyz="0.0 0.0 0.0185" rpy="${pi/2} 0.0 ${pi/2}" />
+      <parent link="rear_bumper_link" />
       <child link="rear_light_link" />
     </joint>

File: panther_description/urdf/components/external_antenna.urdf.xacro (robot description, xacro)
@@ -40,7 +40,7 @@
         <origin xyz="0.045 0.0 0.0058" rpy="0.0 0.0 0.0" />
         <mass value="0.59" />
-        <inertia ixx="0.003964" ixy="0.0" ixz="0.0"
-          iyy="0.0003964" iyz="0.0"
-          izz="0.0004177" />
+        <inertia ixx="0.003964" ixy="0.0000000" ixz="0.0"
+                                iyy="0.0003964" iyz="0.0"
+                                                izz="0.0004177" />
       </inertial>
     </link>
