Commit message: Add reling link (#474)
* Add reling link

* fix

* Typos

* mount link

* Undo

File: husarion_ugv_description/urdf/lynx/base.urdf.xacro (robot description, xacro)
@@ -96,4 +96,10 @@
     </joint>
     <link name="cover_link" />
+    <joint name="cover_to_mount_joint" type="fixed">
+      <origin xyz="0.0 0.0 0.0315" rpy="0.0 0.0 0.0" />
+      <parent link="cover_link" />
+      <child link="mount_link" />
+    </joint>
+    <link name="mount_link" />
   </xacro:macro>
 </robot>

File: husarion_ugv_description/urdf/panther/base.urdf.xacro (robot description, xacro)
@@ -64,9 +64,15 @@
     <link name="lights_channel_2_link" />
     <joint name="base_to_cover_joint" type="fixed">
-      <origin xyz="0.0 0.0 0.1715" rpy="0.0 0.0 0.0" />
+      <origin xyz="0.0 0.0 0.14" rpy="0.0 0.0 0.0" />
       <parent link="base_link" />
       <child link="cover_link" />
     </joint>
     <link name="cover_link" />
+    <joint name="cover_to_mount_joint" type="fixed">
+      <origin xyz="0.0 0.0 0.0315" rpy="0.0 0.0 0.0" />
+      <parent link="cover_link" />
+      <child link="mount_link" />
+    </joint>
+    <link name="mount_link" />
   </xacro:macro>
 </robot>
