Commit message: Ros2 change wheels mount point (#492)
* use wheel mount point instead of wheel separation

* Update Lynx meshes

* fix dimensions

* adjust COM

* review fixes

File: husarion_ugv_description/urdf/common/wheel.urdf.xacro (robot description, xacro)
@@ -2,32 +2,42 @@
 <robot xmlns:xacro="http://wiki.ros.org/xacro">
   <!-- wheel defining macro -->
-  <xacro:macro name="wheel" params="wheel_config wheel_separation_x prefix">
+  <xacro:macro name="wheel" params="config prefix mount_point_x mount_point_y">
     <xacro:if value="${prefix == 'fl'}">
-      <xacro:property name="x" value="${wheel_separation_x/2.0}" />
-      <xacro:property name="y" value="${wheel_config['wheel_separation']/2.0}" />
-      <xacro:property name="inertia_y_offset" value="${wheel_config['inertia_y_offset']}" />
+      <xacro:property name="x" value="${mount_point_x}" />
+      <xacro:property name="y" value="${mount_point_y}" />
+      <xacro:property name="mount_point_offset" value="${config['mount_point_offset']}" />
+      <xacro:property name="inertia_y_offset" value="${config['inertia_y_offset']}" />
       <xacro:property name="fdir" value="1 -1 0" />
     </xacro:if>
     <xacro:if value="${prefix == 'fr'}">
-      <xacro:property name="x" value="${wheel_separation_x/2.0}" />
-      <xacro:property name="y" value="-${wheel_config['wheel_separation']/2.0}" />
-      <xacro:property name="inertia_y_offset" value="${-wheel_config['inertia_y_offset']}" />
+      <xacro:property name="x" value="${mount_point_x}" />
+      <xacro:property name="y" value="-${mount_point_y}" />
+      <xacro:property name="mount_point_offset" value="-${config['mount_point_offset']}" />
+      <xacro:property name="inertia_y_offset" value="${-config['inertia_y_offset']}" />
       <xacro:property name="fdir" value="1 1 0" />
     </xacro:if>
     <xacro:if value="${prefix == 'rl'}">
-      <xacro:property name="x" value="-${wheel_separation_x/2.0}" />
-      <xacro:property name="y" value="${wheel_config['wheel_separation']/2.0}" />
-      <xacro:property name="inertia_y_offset" value="${wheel_config['inertia_y_offset']}" />
+      <xacro:property name="x" value="-${mount_point_x}" />
+      <xacro:property name="y" value="${mount_point_y}" />
+      <xacro:property name="mount_point_offset" value="${config['mount_point_offset']}" />
+      <xacro:property name="inertia_y_offset" value="${config['inertia_y_offset']}" />
       <xacro:property name="fdir" value="1 1 0" />
     </xacro:if>
     <xacro:if value="${prefix == 'rr'}">
-      <xacro:property name="x" value="-${wheel_separation_x/2.0}" />
-      <xacro:property name="y" value="-${wheel_config['wheel_separation']/2.0}" />
-      <xacro:property name="inertia_y_offset" value="${-wheel_config['inertia_y_offset']}" />
+      <xacro:property name="x" value="-${mount_point_x}" />
+      <xacro:property name="y" value="-${mount_point_y}" />
+      <xacro:property name="mount_point_offset" value="-${config['mount_point_offset']}" />
+      <xacro:property name="inertia_y_offset" value="${-config['inertia_y_offset']}" />
       <xacro:property name="fdir" value="1 -1 0" />
     </xacro:if>
+    <joint name="body_to_${prefix}_wheel_base_joint" type="fixed">
+      <origin xyz="${x} ${y} 0.0" rpy="0.0 0.0 0.0" />
+      <parent link="body_link" />
+      <child link="${prefix}_wheel_base_link" />
+    </joint>
+    <link name="${prefix}_wheel_base_link" />
     <joint name="${prefix}_wheel_joint" type="continuous">
-      <origin xyz="${x} ${y} 0.0" rpy="0.0 0.0 0.0" />
-      <parent link="base_link" />
+      <origin xyz="0.0 ${mount_point_offset} 0.0" rpy="0.0 0.0 0.0" />
+      <parent link="${prefix}_wheel_base_link" />
       <child link="${prefix}_wheel_link" />
       <axis xyz="0.0 1.0 0.0" />
@@ -39,5 +49,5 @@
         <origin xyz="0.0 0.0 0.0" rpy="0.0 0.0 0.0" />
         <geometry>
-          <mesh filename="package://${wheel_config['mesh_package']}/${wheel_config['folder_path']}/${prefix}_wheel.dae" />
+          <mesh filename="package://${config['mesh_package']}/${config['folder_path']}/${prefix}_wheel.dae" />
         </geometry>
       </visual>
@@ -45,21 +55,21 @@
         <origin xyz="0.0 0.0 0.0" rpy="-${pi/2} 0.0 0.0" />
         <geometry>
-          <cylinder radius="${wheel_config['wheel_radius']}" length="${wheel_config['wheel_width']}" />
+          <cylinder radius="${config['wheel_radius']}" length="${config['wheel_width']}" />
         </geometry>
       </collision>
       <inertial>
         <origin xyz="0.0 ${inertia_y_offset} 0.0" rpy="0.0 0.0 0.0" />
-        <mass value="${wheel_config['mass']}" />
+        <mass value="${config['mass']}" />
         <inertia
-          ixx="${wheel_config['inertia']['ixx']}"
+          ixx="${config['inertia']['ixx']}"
           ixy="0.0"
           ixz="0.0"
-          iyy="${wheel_config['inertia']['iyy']}"
+          iyy="${config['inertia']['iyy']}"
           iyz="0.0"
-          izz="${wheel_config['inertia']['izz']}" />
+          izz="${config['inertia']['izz']}" />
       </inertial>
     </link>
     <xacro:if value="${use_sim}">
-      <xacro:if value="${wheel_config['mecanum']}">
+      <xacro:if value="${config['mecanum']}">
         <gazebo reference="${prefix}_wheel_link" xmlns:ignition="http://ignitionrobotics.org/schema">
           <collision>

File: husarion_ugv_description/urdf/lynx/base.urdf.xacro (robot description, xacro)
@@ -4,5 +4,11 @@
     name="body"
     params="wheel_radius imu_xyz imu_rpy">
-    <link name="base_link">
+    <joint name="base_to_body_joint" type="fixed">
+      <origin xyz="0.0 0.0 0.0" rpy="0.0 0.0 0.0" />
+      <parent link="base_link" />
+      <child link="body_link" />
+    </joint>
+    <link name="base_link" />
+    <link name="body_link">
       <visual>
         <geometry>
@@ -11,91 +17,37 @@
       </visual>
       <collision>
-        <origin xyz="0.0 0.0 0.09" rpy="0.0 0.0 0.0" />
+        <origin xyz="0.0 0.0 0.0" rpy="0.0 0.0 0.0" />
         <geometry>
-          <!-- TODO change when models ready -->
-          <!-- <mesh filename="package://husarion_ugv_description/meshes/panther/body_collision.stl" /> -->
-          <box size="0.64 0.34 0.28" />
+          <mesh filename="package://husarion_ugv_description/meshes/lynx/base_collision.dae" />
         </geometry>
       </collision>
       <inertial>
-        <origin xyz="0.0 0.0 0.0" rpy="0.0 0.0 0.0" />
-        <mass value="30.0" />
-        <!-- TODO calculate real interia -->
-        <inertia ixx="0.46856"  ixy="0.0"     ixz="0.0"
-                                iyy="1.22285" iyz="0.0"
-                                              izz="1.51185" />
+        <origin xyz="-0.052 0.001 0.038" rpy="0.0 0.0 0.0" />
+        <mass value="30.656" />
+        <inertia ixx="0.6572" ixy="0.0334"  ixz="0.1739"
+                              iyy="1.443"   iyz="0.0082"
+                                            izz="1.598" />
       </inertial>
     </link>
-    <joint name="base_to_footprint_joint" type="fixed">
+    <joint name="body_to_footprint_joint" type="fixed">
       <origin xyz="0.0 0.0 -${wheel_radius}" rpy="0.0 0.0 0.0" />
-      <parent link="base_link" />
+      <parent link="body_link" />
       <child link="base_footprint" />
     </joint>
     <link name="base_footprint" />
-    <joint name="base_to_user_compartment_joint" type="fixed">
-      <origin xyz="0.0 0.0 0.00535" rpy="0.0 0.0 0.0" />
-      <parent link="base_link" />
-      <child link="user_compartment_link" />
-    </joint>
-    <link name="user_compartment_link">
-      <visual>
-        <geometry>
-          <mesh filename="package://husarion_ugv_description/meshes/lynx/user_compartment.dae" />
-        </geometry>
-      </visual>
-      <!-- TODO change when models ready -->
-      <!-- <collision>
-        <geometry>
-          <mesh filename="package://husarion_ugv_description/meshes/panther/user_compartment_collision.stl" />
-        </geometry>
-      </collision> -->
-      <inertial>
-        <!-- TODO calculate real interia -->
-        <mass value="30.0" />
-        <inertia ixx="0.46856"  ixy="0.0"     ixz="0.0"
-                                iyy="1.22285" iyz="0.0"
-                                              izz="1.51185" />
-      </inertial>
-    </link>
-    <joint name="base_to_battery_joint" type="fixed">
-      <origin xyz="-0.2628 -0.07945 0.07265" rpy="0.0 0.0 0.0" />
-      <parent link="base_link" />
-      <child link="battery_link" />
-    </joint>
-    <link name="battery_link">
-      <visual>
-        <geometry>
-          <mesh filename="package://husarion_ugv_description/meshes/lynx/battery.dae" />
-        </geometry>
-      </visual>
-      <!-- TODO change when models ready -->
-      <!-- <collision>
-        <geometry>
-          <mesh filename="package://husarion_ugv_description/meshes/panther/battery_collision.stl" />
-        </geometry>
-      </collision> -->
-      <inertial>
-        <mass value="30.0" />
-        <!-- TODO calculate real interia -->
-        <inertia ixx="0.46856"  ixy="0.0"     ixz="0.0"
-                                iyy="1.22285" iyz="0.0"
-                                              izz="1.51185" />
-      </inertial>
-    </link>
-    <joint name="base_to_imu_joint" type="fixed">
+    <joint name="body_to_imu_joint" type="fixed">
       <origin xyz="${imu_xyz}" rpy="${imu_rpy}" />
-      <parent link="base_link" />
+      <parent link="body_link" />
       <child link="imu_link" />
     </joint>
     <link name="imu_link" />
-    <joint name="base_to_cover_joint" type="fixed">
-      <!-- TODO change to real value -->
-      <origin xyz="0.0 0.0 0.2085" rpy="0.0 0.0 0.0" />
-      <parent link="base_link" />
+    <joint name="body_to_cover_joint" type="fixed">
+      <origin xyz="0.0 0.0 0.2098" rpy="0.0 0.0 0.0" />
+      <parent link="body_link" />
       <child link="cover_link" />
     </joint>
     <link name="cover_link" />
     <joint name="cover_to_mount_joint" type="fixed">
-      <origin xyz="0.0 0.0 0.0315" rpy="0.0 0.0 0.0" />
+      <origin xyz="0.0 0.0 0.0217" rpy="0.0 0.0 0.0" />
       <parent link="cover_link" />
       <child link="mount_link" />

File: husarion_ugv_description/urdf/lynx/lynx_macro.urdf.xacro (robot description, xacro)
@@ -12,5 +12,6 @@
     <xacro:property name="ns" value='${namespace + "/" if namespace else ""}' />
     <xacro:property name="wheel_config" value="${xacro.load_yaml(wheel_config_file)}" />
-    <xacro:property name="wheel_separation_x" value="0.35" />
+    <xacro:property name="wheelbase" value="0.35" />
+    <xacro:property name="wheel_mount_point_y" value="0.1675" />
     <!-- INCLUDE ROBOT PARTS DEFINITIONS -->
     <xacro:include filename="$(find husarion_ugv_description)/urdf/lynx/base.urdf.xacro" ns="body" />
@@ -24,18 +25,22 @@
     <!-- WHEEL DECLARATION -->
     <xacro:wheel.wheel
-      wheel_config="${wheel_config}"
-      wheel_separation_x="${wheel_separation_x}"
+      config="${wheel_config}"
+      mount_point_x="${wheelbase/2.0}"
+      mount_point_y="${wheel_mount_point_y}"
       prefix="fl" />
     <xacro:wheel.wheel
-      wheel_config="${wheel_config}"
-      wheel_separation_x="${wheel_separation_x}"
+      config="${wheel_config}"
+      mount_point_x="${wheelbase/2.0}"
+      mount_point_y="${wheel_mount_point_y}"
       prefix="fr" />
     <xacro:wheel.wheel
-      wheel_config="${wheel_config}"
-      wheel_separation_x="${wheel_separation_x}"
+      config="${wheel_config}"
+      mount_point_x="${wheelbase/2.0}"
+      mount_point_y="${wheel_mount_point_y}"
       prefix="rl" />
     <xacro:wheel.wheel
-      wheel_config="${wheel_config}"
-      wheel_separation_x="${wheel_separation_x}"
+      config="${wheel_config}"
+      mount_point_x="${wheelbase/2.0}"
+      mount_point_y="${wheel_mount_point_y}"
       prefix="rr" />
     <ros2_control name="${ns}lynx_system" type="system">

File: husarion_ugv_description/urdf/panther/base.urdf.xacro (robot description, xacro)
@@ -1,11 +1,15 @@
 <?xml version="1.0" encoding="utf-8"?>
 <robot xmlns:xacro="http://wiki.ros.org/xacro">
-  <!-- body defining macro -->
   <xacro:macro
     name="body"
     params="wheel_radius imu_xyz imu_rpy">
-    <link name="base_link">
+    <joint name="base_to_body_joint" type="fixed">
+      <origin xyz="0.0 0.0 0.0" rpy="0.0 0.0 0.0" />
+      <parent link="base_link" />
+      <child link="body_link" />
+    </joint>
+    <link name="base_link" />
+    <link name="body_link">
       <visual>
-        <origin xyz="0.0 0.0 0.0" rpy="0.0 0.0 0.0" />
         <geometry>
           <mesh filename="package://husarion_ugv_description/meshes/panther/base.dae" />
@@ -19,6 +23,5 @@
       </collision>
       <inertial>
-        <!-- TODO Fix oringin -->
-        <origin xyz="0.0 0.0 0.0" rpy="0.0 0.0 0.0" />
+        <origin xyz="-0.008 0.01 0.029" rpy="0.0 0.0 0.0" />
         <mass value="43.0" />
         <inertia ixx="2.630036" ixy="-0.023480" ixz="0.052320"
@@ -27,19 +30,19 @@
       </inertial>
     </link>
-    <joint name="base_to_footprint_joint" type="fixed">
+    <joint name="body_to_footprint_joint" type="fixed">
       <origin xyz="0.0 0.0 -${wheel_radius}" rpy="0.0 0.0 0.0" />
-      <parent link="base_link" />
+      <parent link="body_link" />
       <child link="base_footprint" />
     </joint>
     <link name="base_footprint" />
-    <joint name="base_to_imu_joint" type="fixed">
+    <joint name="body_to_imu_joint" type="fixed">
       <origin xyz="${imu_xyz}" rpy="${imu_rpy}" />
-      <parent link="base_link" />
+      <parent link="body_link" />
       <child link="imu_link" />
     </joint>
     <link name="imu_link" />
-    <joint name="base_to_front_bumper_joint" type="fixed">
+    <joint name="body_to_front_bumper_joint" type="fixed">
       <origin xyz="0.362 0.0 0.0" rpy="0.0 0.0 0.0" />
-      <parent link="base_link" />
+      <parent link="body_link" />
       <child link="front_bumper_link" />
     </joint>
@@ -51,7 +54,7 @@
     </joint>
     <link name="lights_channel_1_link" />
-    <joint name="base_to_rear_bumper_joint" type="fixed">
+    <joint name="body_to_rear_bumper_joint" type="fixed">
       <origin xyz="-0.362 0.0 0.0" rpy="0.0 0.0 ${pi}" />
-      <parent link="base_link" />
+      <parent link="body_link" />
       <child link="rear_bumper_link" />
     </joint>
@@ -63,7 +66,7 @@
     </joint>
     <link name="lights_channel_2_link" />
-    <joint name="base_to_cover_joint" type="fixed">
+    <joint name="body_to_cover_joint" type="fixed">
       <origin xyz="0.0 0.0 0.14" rpy="0.0 0.0 0.0" />
-      <parent link="base_link" />
+      <parent link="body_link" />
       <child link="cover_link" />
     </joint>

File: husarion_ugv_description/urdf/panther/panther_macro.urdf.xacro (robot description, xacro)
@@ -16,5 +16,6 @@
     <xacro:property name="ns" value='${namespace + "/" if namespace else ""}' />
     <xacro:property name="wheel_config" value="${xacro.load_yaml(wheel_config_file)}" />
-    <xacro:property name="wheel_separation_x" value="0.44" />
+    <xacro:property name="wheelbase" value="0.44" />
+    <xacro:property name="wheel_mount_point_y" value="0.2575" />
     <!-- INCLUDE ROBOT PARTS DEFINITIONS -->
     <xacro:include filename="$(find husarion_ugv_description)/urdf/panther/base.urdf.xacro" ns="body" />
@@ -28,18 +29,22 @@
     <!-- WHEEL DECLARATION -->
     <xacro:wheel.wheel
-      wheel_config="${wheel_config}"
-      wheel_separation_x="${wheel_separation_x}"
+      config="${wheel_config}"
+      mount_point_x="${wheelbase/2.0}"
+      mount_point_y="${wheel_mount_point_y}"
       prefix="fl" />
     <xacro:wheel.wheel
-      wheel_config="${wheel_config}"
-      wheel_separation_x="${wheel_separation_x}"
+      config="${wheel_config}"
+      mount_point_x="${wheelbase/2.0}"
+      mount_point_y="${wheel_mount_point_y}"
       prefix="fr" />
     <xacro:wheel.wheel
-      wheel_config="${wheel_config}"
-      wheel_separation_x="${wheel_separation_x}"
+      config="${wheel_config}"
+      mount_point_x="${wheelbase/2.0}"
+      mount_point_y="${wheel_mount_point_y}"
       prefix="rl" />
     <xacro:wheel.wheel
-      wheel_config="${wheel_config}"
-      wheel_separation_x="${wheel_separation_x}"
+      config="${wheel_config}"
+      mount_point_x="${wheelbase/2.0}"
+      mount_point_y="${wheel_mount_point_y}"
       prefix="rr" />
     <ros2_control name="${ns}panther_system" type="system">
