Commit message: fix Lynx imu default position (#515)

File: husarion_ugv_description/urdf/lynx.urdf.xacro (robot description, xacro)
@@ -2,6 +2,5 @@
 <robot name="lynx" xmlns:xacro="http://wiki.ros.org/xacro">
   <xacro:arg name="use_sim" default="false" />
-  <!-- TODO find IMU position -->
-  <xacro:arg name="imu_xyz" default="0.169 0.025 0.092" />
+  <xacro:arg name="imu_xyz" default="0.052 0.073 -0.006" />
   <xacro:arg name="imu_rpy" default="0.0 0.0 -1.57" />
   <xacro:arg name="wheel_config_file"

File: husarion_ugv_description/urdf/lynx/lynx_macro.urdf.xacro (robot description, xacro)
@@ -7,7 +7,11 @@
             battery_config_file
             use_sim:=false
-            imu_xyz:='0.169 0.025 0.092'
+            imu_xyz:='0.052 0.073 -0.006'
             imu_rpy:='0.0 0.0 -1.57'
             namespace:=''">
+    <xacro:if value="${use_sim}">
+      <xacro:property name="imu_xyz" value="0.052 0.073 -0.006" />
+      <xacro:property name="imu_rpy" value="0.0 0.0 -1.57" />
+    </xacro:if>
     <xacro:property name="ns" value='${namespace + "/" if namespace else ""}' />
     <xacro:property name="wheel_config" value="${xacro.load_yaml(wheel_config_file)}" />
